Commit message: Updated urdf and moveit_config package

File: ur5_qb_description/urdf/ur5_qb.xacro (robot description, xacro)
@@ -9,26 +9,27 @@
 	<xacro:arg name="namespace" default="qbhand"/>
     <link name="world" />
-	<link name="table" />
-	<link name="camera_frame">
+	<!-- <link name="table" /> -->
+	<!-- <link name="camera_frame">
 		<visual>
 			<geometry>
-				<box size="0.5 1 1"/>
+				<box size="0.25 0.5 0.5"/>
 			</geometry>
 		</visual>
 		<collision>
 			<geometry>
-				<box size="0.5 1 1"/>
+				<box size="0.25 0.5 0.5"/>
 			</geometry>
 		</collision>
 	</link>
+ -->
 	<xacro:build_hand_from_yaml configuration="qbhand_left" namespace="$(arg namespace)" parent="ee">
 		<origin xyz="0 0 0" rpy="0 1.57 0"/>
 	</xacro:build_hand_from_yaml>
-	<joint name="world_to_table" type="fixed">
+	<joint name="world_to_robot" type="fixed">
 		<parent link="world" />
-		<child link = "table" />
-		<origin xyz="0 0 0.25" rpy="0.0 0.0 0.0" />
+		<child link = "base_link" />
+		<origin xyz="0 0 0.5" rpy="0.0 0.0 0.0" />
 	</joint>
-	<joint name="world_to_camera" type="fixed">
+<!-- 	<joint name="world_to_camera" type="fixed">
 		<parent link="world" />
 		<child link = "camera_frame" />
@@ -39,5 +40,5 @@
 		<child link = "base_link" />
 		<origin xyz="0.0 0.0 0" rpy="0.0 0.0 0.0" />
-	</joint>
+	</joint> -->
 <!-- 	<joint name="ur5_to_qb" type="revolute">
 		 <axis xyz="0 0 1"/>

Commit message: Moveit config files.

File: ur5_qb_description/urdf/ur5_qb.xacro (robot description, xacro)
@@ -7,44 +7,49 @@
     transmission_hw_interface="$(arg transmission_hw_interface)"  />
   <xacro:include filename="$(find qb_hand_description)/urdf/qbhand.utils.xacro"/>
-	<xacro:arg name="namespace" default="qbhand"/>
-    <link name="world" />
-	<!-- <link name="table" /> -->
-	<!-- <link name="camera_frame">
-		<visual>
-			<geometry>
-				<box size="0.25 0.5 0.5"/>
-			</geometry>
-		</visual>
-		<collision>
-			<geometry>
-				<box size="0.25 0.5 0.5"/>
-			</geometry>
-		</collision>
-	</link>
- -->
-	<xacro:build_hand_from_yaml configuration="qbhand_left" namespace="$(arg namespace)" parent="ee">
-		<origin xyz="0 0 0" rpy="0 1.57 0"/>
-	</xacro:build_hand_from_yaml>
-	<joint name="world_to_robot" type="fixed">
-		<parent link="world" />
-		<child link = "base_link" />
-		<origin xyz="0 0 0.5" rpy="0.0 0.0 0.0" />
-	</joint>
-<!-- 	<joint name="world_to_camera" type="fixed">
-		<parent link="world" />
-		<child link = "camera_frame" />
-		<origin xyz="0.0 0.0 0" rpy="0.0 1.571 0.0" />
-	</joint>
-	<joint name="table_to_robot" type="fixed">
-		<parent link="table" />
-		<child link = "base_link" />
-		<origin xyz="0.0 0.0 0" rpy="0.0 0.0 0.0" />
-	</joint> -->
-<!-- 	<joint name="ur5_to_qb" type="revolute">
-		 <axis xyz="0 0 1"/>
-   	    <limit effort="1000.0" lower="-6.28" upper="6.28" velocity="0.5"/>
-		<parent link="ee_link" />
-		<child link = "qbhand1_base_link" />
-		<origin xyz="0.0 0.0 0" rpy="0.0 0.0 0.0" />
-	</joint> -->
+  <xacro:arg name="namespace" default="qbhand"/>
+  <link name="world" />
+<!--
+  <link name="table" />
+  <link name="camera_frame">
+    <visual>
+      <geometry>
+        <box size="0.25 0.5 0.5"/>
+      </geometry>
+    </visual>
+    <collision>
+      <geometry>
+        <box size="0.25 0.5 0.5"/>
+      </geometry>
+    </collision>
+  </link>
+-->
+  <xacro:build_hand_from_yaml configuration="qbhand_left" namespace="$(arg namespace)" parent="ee">
+    <origin xyz="0 0 0" rpy="0 1.57 0"/>
+  </xacro:build_hand_from_yaml>
+  <joint name="world_to_robot" type="fixed">
+    <parent link="world" />
+    <child link = "base_link" />
+  <origin xyz="0 0 0.5" rpy="0.0 0.0 0.0" />
+  </joint>
+<!--
+  <joint name="world_to_camera" type="fixed">
+    <parent link="world" />
+    <child link = "camera_frame" />
+    <origin xyz="0.0 0.0 0" rpy="0.0 1.571 0.0" />
+  </joint>
+  <joint name="table_to_robot" type="fixed">
+    <parent link="table" />
+    <child link = "base_link" />
+    <origin xyz="0.0 0.0 0" rpy="0.0 0.0 0.0" />
+  </joint>
+-->
+<!--
+  <joint name="ur5_to_qb" type="revolute">
+    <axis xyz="0 0 1"/>
+    <limit effort="1000.0" lower="-6.28" upper="6.28" velocity="0.5"/>
+    <parent link="ee_link" />
+    <child link = "qbhand1_base_link" />
+    <origin xyz="0.0 0.0 0" rpy="0.0 0.0 0.0" />
+  </joint>
+-->
 </robot>

Commit message: Added moveit and gazebo launch

File: ur5_qb_description/urdf/ur5_qb.xacro (robot description, xacro)
@@ -9,18 +9,4 @@
 	<xacro:arg name="namespace" default="qbhand"/>
     <link name="world" />
-	<!-- <link name="table" /> -->
-	<!-- <link name="camera_frame">
-		<visual>
-			<geometry>
-				<box size="0.25 0.5 0.5"/>
-			</geometry>
-		</visual>
-		<collision>
-			<geometry>
-				<box size="0.25 0.5 0.5"/>
-			</geometry>
-		</collision>
-	</link>
- -->
 	<xacro:build_hand_from_yaml configuration="qbhand_left" namespace="$(arg namespace)" parent="ee">
 		<origin xyz="0 0 0" rpy="0 1.57 0"/>
@@ -31,20 +17,3 @@
 		<origin xyz="0 0 0.5" rpy="0.0 0.0 0.0" />
 	</joint>
-<!-- 	<joint name="world_to_camera" type="fixed">
-		<parent link="world" />
-		<child link = "camera_frame" />
-		<origin xyz="0.0 0.0 0" rpy="0.0 1.571 0.0" />
-	</joint>
-	<joint name="table_to_robot" type="fixed">
-		<parent link="table" />
-		<child link = "base_link" />
-		<origin xyz="0.0 0.0 0" rpy="0.0 0.0 0.0" />
-	</joint> -->
-<!-- 	<joint name="ur5_to_qb" type="revolute">
-		 <axis xyz="0 0 1"/>
-   	    <limit effort="1000.0" lower="-6.28" upper="6.28" velocity="0.5"/>
-		<parent link="ee_link" />
-		<child link = "qbhand1_base_link" />
-		<origin xyz="0.0 0.0 0" rpy="0.0 0.0 0.0" />
-	</joint> -->
 </robot>

File: ur_description/urdf/ur5_robot.urdf.xacro (robot description, xacro)
@@ -11,15 +11,9 @@
     transmission_hw_interface="$(arg transmission_hw_interface)"
   />
-  <!-- qbsofthand -->
- <!-- <xacro:include filename="$(find ur_description)/urdf/qbhand.utils.xacro"/>
   <link name="world" />
   <joint name="world_joint" type="fixed">
     <parent link="world" />
     <child link = "base_link" />
-    <origin xyz="0.0 0.0 0.0" rpy="0.0 0.0 0.0" />
+    <origin xyz="0.0 0.0 0.5" rpy="0.0 0.0 0.0" />
   </joint>
-	<link name="ee_qb"/>
-	<xacro:build_hand_from_yaml configuration="qbhand_right" namespace="$(arg namespace)" parent="ee_link">
-		<origin xyz="0 0 0" rpy="0 0 0"/>
-	</xacro:build_hand_from_yaml> -->
 </robot>
