Commit message: Solved Gazebo import error

File: ur5_qb_description/urdf/ur5_qb_new.urdf.xacro (robot description, xacro)
@@ -2,15 +2,17 @@
 <robot xmlns:xacro="http://wiki.ros.org/xacro" name="ur5_qb_new" >
   <xacro:include filename="$(find ur_description)/urdf/ur5.urdf.xacro" />
-  <link name="world" />
-  <xacro:arg name="initial_z" default="1.0"/>
-	<joint name="world_to_robot" type="fixed">
+  <xacro:ur5_robot prefix="ur_" joint_limited="false"/>
+  <!-- <xacro:arg name="initial_z" default="1.0"/> -->
+    <link name = "world" />
+    <!-- <link name="dummy_base" /> -->
+	<joint name="dummy_link" type="fixed">
 		<parent link="world" />
 		<child link = "ur_base_link" />
-		<origin xyz="0 0 $(arg initial_z)" rpy="0.0 0.0 0.0" />
+		<origin xyz="0 0 1.0" rpy="0.0 0.0 0.0" />
 	</joint>
-	<xacro:ur5_robot prefix="ur_" joint_limited="false"/>
   <gazebo>
    <plugin name="gazebo_ros_control" filename="libgazebo_ros_control.so">
-    <!-- <robotNamespace>ur5_qb_new</robotNamespace> -->
+    <robotNamespace>ur5_qb_new</robotNamespace>
+    <legacyModeNS>true</legacyModeNS>
   </plugin>
   </gazebo>
